Commit message: Updated ROS

File: src/semesterprosjekt/urdf/boat_arm.xacro (robot description, xacro)
@@ -6,84 +6,47 @@
     <static>true</static>
   </gazebo> -->
- <!-- <xacro:property name="density" value="1" /> -->
   <material name="COLOR">
-   <color rgba="1 1 1 1"/>
- </material>
-  <link name='base_link'>
-    <pose>0 0 0.1 0 0 0</pose>
-    <visual name='chassis_visual'>
-      <origin xyz="0 0 -0.1" rpy="0 0 ${pi/2}"/>
+     <color rgba="1 1 1 1"/>
+   </material>
+    <link name='base_link'>
+      <pose>0 0 ${-(0.221/2) + (0.05/2)} 0 0 0</pose>
+      <visual name='chassis_visual'>
+        <origin xyz="${1/2} ${0.4/2} ${-(0.221/2)}" rpy="0 0 ${pi/2}"/>
+        <geometry>
+          <mesh filename="package://semesterprosjekt/mesh/Bote.stl" scale="0.001 0.001 0.001"/>
+        </geometry>
+        <material name="COLOR"/>
+      </visual>
+      <collision>
+        <origin xyz="0 0 0" rpy="0 0 0"/>
+        <geometry>0.07
+          <box size="1 0.3 0.221"/>
+        </geometry>
+      </collision>
+      <inertial>
+        <mass value="30"/>
+        <inertia ixx="0.1075" ixy="0.0" ixz="0.0" iyy="10.0008" iyz="0.0" izz="10.0075"/>
+      </inertial>
+  </link>
+  <link name='front_ball'>
+    <collision>
       <geometry>
-        <mesh filename="package://semesterprosjekt/mesh/RobotBatPOrsjekt_v4_v5.stl" scale="0.001 0.001 0.001"/>
-       <!-- <box size="1 0.3 0.1"/> -->
-      </geometry>
-      <material name="COLOR"/>
-    </visual>
-    <collision>
-      <origin xyz="0 0 0.07" rpy="0 0 0"/>
-      <geometry>
-        <!-- <box size="1 0.4 0.1"/> -->
-        <box size="1 0.4 0.1"/>
-      </geometry>
-    </collision>
-    <inertial>
-      <mass value="10"/>
-      <inertia ixx="0.1075" ixy="0.0" ixz="0.0" iyy="10.0008" iyz="0.0" izz="10.0075"/>
-    </inertial>
-</link>
-  <link name='left_thruster'>
-    <visual>
-      <geometry>
-       <cylinder length="0.07" radius="0.03"/>
+       <sphere radius="0.05"/>
      </geometry>
-     <!-- <origin rpy="1.5707963 0 0" xyz="0.15 0.465 -0.03"/> -->
-     <origin rpy="${pi/2} 0 ${pi/2}" xyz="-0.465 0.15 -0.03"/>
-   </visual>
+     <origin rpy="0 0 0" xyz="0 0 0"/>
+   </collision>
+   <inertial>
+     <mass value="0.01"/>
+     <inertia ixx="0.1075" ixy="0.0" ixz="0.0" iyy="0.0008" iyz="0.0" izz="0.0075"/>
+   </inertial>
   </link>
-  <link name='right_thruster'>
-    <visual>
-      <geometry>
-       <cylinder length="0.07" radius="0.03"/>
-     </geometry>
-     <!-- <origin rpy="1.5707963 0 0" xyz="-0.15 0.465 -0.03"/> -->
-     <origin rpy="${pi/2} 0 ${pi/2}" xyz="-0.465 -0.15 -0.03"/>
-   </visual>
-  </link>
-  <joint name="base_to_left_thruster" type="fixed">
-    <parent link="base_link"/>
-    <child link="left_thruster"/>
-  </joint>
-  <joint name="base_to_right_thruster" type="fixed">
-    <parent link="base_link"/>
-    <child link="right_thruster"/>
-  </joint>
-  <joint name="left_front_wheel_j" type="continuous">
-    <origin xyz="0.20 0.20 0" rpy="${-pi/2} 0 0"/>
-    <parent link="base_link"/>
-    <child link="lf_wheel"/>
-    <axis xyz="0 0 1" rpy="0 0 0"/>
-    <limit effort="100" velocity="100"/>
-  </joint>
-  <xacro:link_wheel link_name="lf_wheel">
-    <!-- collison -->
-    <origin xyz="0 0 0" rpy="0 0 0"/>
-    <!-- inertia -->
-    <origin xyz="0 0 0" rpy="0 0 0"/>
-  </xacro:link_wheel>
-  <joint name="right_front_wheel_j" type="continuous">
-    <origin xyz="0.20 -0.20 0" rpy="${-pi/2} 0 0"/>
-    <parent link="base_link"/>
-    <child link="rf_wheel"/>
-    <axis xyz="0 0 1" rpy="0 0 0"/>
-    <limit effort="100" velocity="100"/>
-  </joint>
-  <xacro:link_wheel link_name="rf_wheel">
-    <!-- collison -->
-    <origin xyz="0 0 0" rpy="0 0 0"/>
-    <!-- inertia -->
-    <origin xyz="0 0 0" rpy="0 0 0"/>
-  </xacro:link_wheel>
+  <joint name="front_ball_j" type="continuous">
+    <origin xyz="0.3 0 ${-(0.221/2)+(0.05/2)}" rpy="0 0 0"/>
+    <parent link="base_link"/>
+    <child link="front_ball"/>
+    <axis xyz="1 1 1" rpy="1 1 1"/>
+  </joint>
   <joint name="left_rear_wheel_j" type="continuous">
-    <origin xyz="-0.20 0.20 0" rpy="${-pi/2} 0 0"/>
+    <origin xyz="-0.20 0.20 ${-(0.221/2)+0.10-(0.05/2)}" rpy="${-pi/2} 0 0"/>
     <parent link="base_link"/>
     <child link="lr_wheel"/>
@@ -98,5 +61,5 @@
   </xacro:link_wheel>
   <joint name="right_rear_wheel_j" type="continuous">
-    <origin xyz="-0.20 -0.20 0" rpy="${-pi/2} 0 0"/>
+    <origin xyz="-0.20 -0.20 ${-(0.221/2)+0.10-(0.05/2)}" rpy="${-pi/2} 0 0"/>
     <parent link="base_link"/>
     <child link="rr_wheel"/>
@@ -110,4 +73,37 @@
     <origin xyz="0 0 0" rpy="0 0 0"/>
   </xacro:link_wheel>
+  <!--############################### -->
+  <!-- SENSORS-->
+  <!--############################### -->
+  <!-- CAMERA-->
+  <!-- ==================================== -->
+  <joint name="camera_joint" type="fixed">
+    <parent link="base_link"/>
+    <child link="camera_link" />
+    <origin xyz="-${(1/2) - (0.01 + 0.025)} 0 ${(0.221/2) + 0.2944}" rpy="0 0 0"/>
+  </joint>
+  <xacro:link_box link_name="camera_link" length="0.05" width="0.07" height="0.02" density="1" mesh_name="nofile">
+    <!-- origin visual -->
+    <origin xyz="0 0 0" rpy="0 0 0"/>
+    <!-- origin collision -->
+    <origin xyz="0 0 0" rpy="0 0 0"/>
+    <!-- origin interia -->
+    <origin xyz="0 0 0" rpy="0 0 0"/>
+  </xacro:link_box>
+  <!-- GPS-->
+  <!-- ==================================== -->
+  <joint name="gps_joint" type="fixed">
+    <parent link="base_link"/>
+    <child link="gps_link" />
+    <origin xyz="-${(1/2) - (0.01 + 0.025)} 0 ${(0.221/2) + 0.3275}" rpy="0 0 0"/>
+  </joint>
+  <xacro:link_sphere link_name="gps_link" radius="0.02" density="1" mesh_name="nofile">
+    <!-- origin visual -->
+    <origin xyz="0 0 ${0.02/2}" rpy="0 0 0"/>
+    <!-- origin collision -->
+    <origin xyz="0 0 0" rpy="0 0 0"/>
+    <!-- origin interia -->
+    <origin xyz="0 0 0" rpy="0 0 0"/>
+  </xacro:link_sphere>
   <!--############################### -->
   <!-- ROBOTIC ARM -->
@@ -116,5 +112,5 @@
   <!-- ==================================== -->
   <joint type="revolute" name="arm_base_joint">
-    <origin xyz="0.05 0 0.18" rpy="0 0 0"/>
+    <origin xyz="${0.500-0.263} 0 ${0.221/2}" rpy="0 0 0"/>
     <child link="arm_base_link"/>
     <parent link="base_link"/>
@@ -149,9 +145,9 @@
     <limit effort="100" velocity="100" lower="-${pi}" upper="${pi}"/>
   </joint>
-  <xacro:link_cylinder link_name="link_1_link" radius="${0.10/2}" length="0.10" density="1"  >
-    <!-- origin visual -->
-    <origin xyz="0 0 0" rpy="-${pi} 0 0"/>
-    <!-- origin collision -->
-    <origin xyz="0 0 0" rpy="0 0 0"/>
+  <xacro:link_cylinder link_name="link_1_link" radius="${0.10/2}" length="0.12" density="1" mesh_name="package://semesterprosjekt/mesh/Robot_Arm_F1_350mm.stl"  >
+    <!-- origin visual -->
+    <origin xyz="0 0 0" rpy="0 0 -${pi/2}"/>
+    <!-- origin collision -->
+    <origin xyz="0 0 -0.04" rpy="0 0 0"/>
     <!-- origin interia -->
     <origin xyz="0 0 0" rpy="0 0 0"/>
@@ -170,15 +166,15 @@
   <!-- ==================================== -->
   <joint type="revolute" name="link_2_joint">
-    <origin xyz="0 -${0.40/2} 0" rpy="${pi/2} 0 0"/>
+    <origin xyz="0 -0.350 0" rpy="${pi/2} 0 0"/>
     <child link="link_2_link"/>
     <parent link="link_1_link"/>
     <axis xyz="0 0 1" rpy="0 0 0"/>
-    <limit effort="100" velocity="100" lower="-${pi/2}" upper="${pi/2}"/>
-  </joint>
-  <xacro:link_cylinder link_name="link_2_link" radius="${0.10/2}" length="0.40" density="1">
-    <!-- origin visual -->
-    <origin xyz="0 0 0" rpy="0 0 0 "/>
-    <!-- origin collision -->
-    <origin xyz="0 0 0" rpy="0 0 0"/>
+    <limit effort="100" velocity="100" lower="-${pi}" upper="${pi}"/>
+  </joint>
+  <xacro:link_cylinder link_name="link_2_link" radius="${0.06/2}" length="${0.350+0.100}" density="1" mesh_name="package://semesterprosjekt/mesh/Robot_Arm_F2_100mm.stl">
+    <!-- origin visual -->
+    <origin xyz="0 0 0" rpy="0 0 ${pi/2}"/>
+    <!-- origin collision -->
+    <origin xyz="0 0 -${0.35/2}" rpy="0 0 0"/>
     <!-- origin interia -->
     <origin xyz="0 0 0" rpy="0 0 0"/>
@@ -197,5 +193,5 @@
   <!-- ==================================== -->
   <joint type="revolute" name="link_3_joint">
-    <origin xyz="0 0 ${0.40/2}" rpy="-${pi/2} 0 0"/>
+    <origin xyz="0 -0.088 0.100" rpy="-${pi/2} 0 0"/>
     <child link="link_3_link"/>
     <parent link="link_2_link"/>
@@ -203,9 +199,9 @@
     <limit effort="100" velocity="100" lower="-${pi}" upper="${pi}"/>
   </joint>
-  <xacro:link_cylinder link_name="link_3_link" radius="${0.10/2}" length="0.10" density="1" >
-    <!-- origin visual -->
-    <origin xyz="0 0 0" rpy="0 0 0"/>
-    <!-- origin collision -->
-    <origin xyz="0 0 0" rpy="0 0 0"/>
+  <xacro:link_cylinder link_name="link_3_link" radius="${0.10/2}" length="0.14" density="1" mesh_name="package://semesterprosjekt/mesh/Robot_Arm_F3_150mm.stl">
+    <!-- origin visual -->
+    <origin xyz="0 0 0" rpy="${pi} 0 -${pi/2}"/>
+    <!-- origin collision -->
+    <origin xyz="0 0 0.05" rpy="0 0 0"/>
     <!-- origin interia -->
     <origin xyz="0 0 0" rpy="0 0 0"/>
@@ -224,15 +220,15 @@
   <!-- ==================================== -->
   <joint type="revolute" name="link_4_joint">
-    <origin xyz="0 -${0.20/2} 0" rpy="${pi/2} 0 0"/>
+    <origin xyz="0 -0.150 0" rpy="${pi/2} 0 0"/>
     <child link="link_4_link"/>
     <parent link="link_3_link"/>
     <axis xyz="0 0 1" rpy="0 0 0"/>
-    <limit effort="100" velocity="100" lower="-${pi/2}" upper="${pi/2}"/>
-  </joint>
-  <xacro:link_cylinder link_name="link_4_link" radius="${0.10/2}" length="0.20" density="1" >
-    <!-- origin visual -->
-    <origin xyz="0 0 0" rpy="0 0 0"/>
-    <!-- origin collision -->
-    <origin xyz="0 0 0" rpy="0 0 0"/>
+    <limit effort="100" velocity="100" lower="-${pi}" upper="${pi}"/>
+  </joint>
+  <xacro:link_cylinder link_name="link_4_link" radius="${0.06/2}" length="0.12" density="1" mesh_name="package://semesterprosjekt/mesh/Robot_Arm_F4_100mm.stl">
+    <!-- origin visual -->
+    <origin xyz="0 0 0" rpy="0 0 -${pi/2}"/>
+    <!-- origin collision -->
+    <origin xyz="0 0 -0.05" rpy="0 0 0"/>
     <!-- origin interia -->
     <origin xyz="0 0 0" rpy="0 0 0"/>
@@ -251,5 +247,5 @@
   <!-- ==================================== -->
   <joint type="revolute" name="link_5_joint">
-    <origin xyz="0 0 0.10" rpy="-${pi/2} 0 0"/>
+    <origin xyz="0 0.088 0.100" rpy="-${pi/2} 0 0"/>
     <child link="link_5_link"/>
     <parent link="link_4_link"/>
@@ -257,9 +253,9 @@
     <limit effort="100" velocity="100" lower="-${pi}" upper="${pi}"/>
   </joint>
-  <xacro:link_cylinder link_name="link_5_link" radius="${0.10/2}" length="0.10" density="1" >
-    <!-- origin visual -->
-    <origin xyz="0 0 0" rpy="0 0 0"/>
-    <!-- origin collision -->
-    <origin xyz="0 0 0" rpy="0 0 0"/>
+  <xacro:link_cylinder link_name="link_5_link" radius="${0.10/2}" length="0.14" density="1" mesh_name="package://semesterprosjekt/mesh/Robot_Arm_F5V_80mm.stl">
+    <!-- origin visual -->
+    <origin xyz="0 0 0" rpy="${pi} 0 ${pi/2}"/>
+    <!-- origin collision -->
+    <origin xyz="0 0 -0.04" rpy="0 0 0"/>
     <!-- origin interia -->
     <origin xyz="0 0 0" rpy="0 0 0"/>
@@ -275,3 +271,30 @@
     </actuator>
   </transmission>
+  <!-- LINK 6 -->
+  <!-- ==================================== -->
+  <joint type="revolute" name="link_6_joint">
+    <origin xyz="0 -${(0.03 + 0.18)/2} 0" rpy="${pi/2} 0 0"/>
+    <child link="link_6_link"/>
+    <parent link="link_5_link"/>
+    <axis xyz="0 0 1" rpy="0 0 0"/>
+    <limit effort="100" velocity="100" lower="-${pi}" upper="${pi}"/>
+  </joint>
+  <xacro:link_cylinder link_name="link_6_link" radius="0.085" length="0.01" density="1" mesh_name="package://semesterprosjekt/mesh/Robot_Arm_Endefector_01.stl">
+    <!-- origin visual -->
+    <origin xyz="0 0 0" rpy="-${pi} 0 0"/>
+    <!-- origin collision -->
+    <origin xyz="0 0 0.09" rpy="-${pi/2} 0 0"/>
+    <!-- origin interia -->
+    <origin xyz="0 0 0" rpy="0 0 0"/>
+  </xacro:link_cylinder>
+  <transmission name="joint_6_trans">
+    <type>transmission_interface/SimpleTransmission</type>
+    <joint name="link_6_joint">
+      <hardwareInterface>hardware_interface/PositionJointInterface</hardwareInterface>
+    </joint>
+    <actuator name="joint_6_motor">
+      <hardwareInterface>hardware_interface/PositionJointInterface</hardwareInterface>
+      <mechanicalReduction>1</mechanicalReduction>
+    </actuator>
+  </transmission>
 </robot>

File: src/semesterprosjekt/urdf/common_macros.xacro (robot description, xacro)
@@ -100,5 +100,5 @@
     </link>
   </xacro:macro>
-  <xacro:macro name="link_wheel" params="link_name length:=0.05 radius:=0.10 density:=15 *origin_col *origin_inertial">
+  <xacro:macro name="link_wheel" params="link_name length:=0.10 radius:=0.10 density:=20 *origin_col *origin_inertial">
     <xacro:property name="mass" value="${pi*length*pow(radius,2)*density}" />
     <link name="${link_name}">
